File: as3320-BandPass-Dev1.sch (EAGLE design)
At the start: 86 parts, among them IC1 CEM3320, IC2 TL074D, IC3 LM4040 5.0V, IC4 TL074D, IC5 TL072D

Commit message: Added 2nd output
Parts:
- added OUTPUT2: PJ301_THONKICONN6, og-pj301_variations:PJ301_THONKICONN6
- added R10: 100K, Pure VCF:GMSN_R-US_M0805
- renumbered IN_MIX to INPUT_MIX, RES-2 to RES, V-OCT1 to V-OCT
Connections:
- removed net N$4: OUTPUTLEVEL.2, R57.1
- new net N$10: IC5B.-IN, IC5B.OUT
- new net N$11: IC5B.+IN, OUTPUTLEVEL.2, R57.1
- new net N$14: R10.1
- new net O1: OUTPUT2.3, R10.2
- net GND: now also OUTPUT2.1
- net N$1: no longer IC5A.OUT
- net N$2: no longer IC5A.-IN
- net N$7: no longer IC5A.+IN
Changed lines of the file:
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@@
 <part name="GND29" library="SparkFun" deviceset="GND" device=""/>
 <part name="R57" library="Pure VCF" deviceset="GMSN_R-US_" device="M0805" value="100K"/>
-<part name="V-OCT1" library="og-pj301_variations" deviceset="PJ301_THONKICONN" device="6"/>
+<part name="V-OCT" library="og-pj301_variations" deviceset="PJ301_THONKICONN" device="6"/>
 <part name="GND1" library="SparkFun" deviceset="GND" device=""/>
 <part name="FREQUENCY" library="og-pots" deviceset="POT_US" device="VERTICAL" value="10kB"/>
@@
 <attribute name="RS-PART" value="828-1783"/>
 </part>
-<part name="RES-2" library="og-pj301_variations" deviceset="PJ301_THONKICONN" device="6"/>
+<part name="RES" library="og-pj301_variations" deviceset="PJ301_THONKICONN" device="6"/>
 <part name="GND5" library="SparkFun" deviceset="GND" device=""/>
 <part name="R71" library="GMSN" deviceset="R-US_" device="R0805" value="100k"/>
@@
 <part name="C32" library="rcl" library_urn="urn:adsk.eagle:library:334" deviceset="C-US" device="C0805K" package3d_urn="urn:adsk.eagle:package:23681/2" value="100n"/>
 <part name="IN_GAIN" library="GMSN" deviceset="9MMPOT" device="" value="9MMPOT"/>
-<part name="IN_MIX" library="og-pj301_variations" deviceset="PJ301_THONKICONN" device="6"/>
+<part name="INPUT_MIX" library="og-pj301_variations" deviceset="PJ301_THONKICONN" device="6"/>
 <part name="R79" library="Pure VCF" deviceset="GMSN_R-US_" device="M0805" value="100"/>
 <part name="GND3" library="SparkFun" deviceset="GND" device=""/>
@@
 <part name="GND6" library="SparkFun" deviceset="GND" device=""/>
 <part name="D2" library="diode" deviceset="DIODE-" device="SOD123" value="1N5819HW"/>
+<part name="OUTPUT2" library="og-pj301_variations" deviceset="PJ301_THONKICONN" device="6"/>
+<part name="GND7" library="SparkFun" deviceset="GND" device=""/>
+<part name="R10" library="Pure VCF" deviceset="GMSN_R-US_" device="M0805" value="100K"/>
 </parts>
 <sheets>
@@
 <instances>
 <instance part="IC2" gate="P" x="35.56" y="165.1" smashed="yes"/>
-<instance part="V-OCT1" gate="G$1" x="71.12" y="27.94" smashed="yes" rot="MR0">
+<instance part="V-OCT" gate="G$1" x="71.12" y="27.94" smashed="yes" rot="MR0">
 <attribute name="NAME" x="73.66" y="32.004" size="1.778" layer="95" rot="MR0"/>
 </instance>
@@
 </instance>
 <instance part="IC4" gate="P" x="25.4" y="165.1" smashed="yes"/>
-<instance part="RES-2" gate="G$1" x="228.6" y="10.16" smashed="yes" rot="MR0">
+<instance part="RES" gate="G$1" x="228.6" y="10.16" smashed="yes" rot="MR0">
 <attribute name="NAME" x="231.14" y="14.224" size="1.778" layer="95" rot="MR0"/>
 </instance>
@@
 <attribute name="VALUE" x="347.98" y="149.86" size="1.778" layer="96" rot="MR180"/>
 </instance>
-<instance part="IN_MIX" gate="G$1" x="378.46" y="142.24" smashed="yes">
+<instance part="INPUT_MIX" gate="G$1" x="378.46" y="142.24" smashed="yes">
 <attribute name="NAME" x="375.92" y="146.304" size="1.778" layer="95"/>
 </instance>
@@
 <attribute name="NAME" x="132.08" y="59.055" size="1.778" layer="95"/>
 <attribute name="VALUE" x="132.08" y="50.8" size="1.778" layer="96"/>
-</instance>
-<instance part="IC5" gate="A" x="48.26" y="-5.08" smashed="yes">
-<attribute name="NAME" x="50.8" y="-8.255" size="1.778" layer="95" rot="MR180"/>
-<attribute name="VALUE" x="50.8" y="0" size="1.778" layer="96" rot="MR180"/>
 </instance>
 <instance part="R6" gate="G$1" x="45.72" y="10.16" smashed="yes">
@@
 <net name="GND" class="1">
 <segment>
-<pinref part="V-OCT1" gate="G$1" pin="1"/>
+<pinref part="V-OCT" gate="G$1" pin="1"/>
 <wire x1="76.2" y1="25.4" x2="78.74" y2="25.4" width="0.1524" layer="91"/>
 <pinref part="GND1" gate="1" pin="GND"/>
 <wire x1="78.74" y1="25.4" x2="78.74" y2="22.86" width="0.1524" layer="91"/>
-<pinref part="V-OCT1" gate="G$1" pin="2"/>
+<pinref part="V-OCT" gate="G$1" pin="2"/>
 <wire x1="76.2" y1="27.94" x2="78.74" y2="27.94" width="0.1524" layer="91"/>
 <wire x1="78.74" y1="27.94" x2="78.74" y2="25.4" width="0.1524" layer="91"/>
@@
 </segment>
 <segment>
-<pinref part="RES-2" gate="G$1" pin="1"/>
+<pinref part="RES" gate="G$1" pin="1"/>
 <wire x1="233.68" y1="7.62" x2="236.22" y2="7.62" width="0.1524" layer="91"/>
 <pinref part="GND5" gate="1" pin="GND"/>
@@
 </segment>
 <segment>
-<pinref part="IN_MIX" gate="G$1" pin="1"/>
+<pinref part="INPUT_MIX" gate="G$1" pin="1"/>
 <wire x1="373.38" y1="139.7" x2="360.68" y2="139.7" width="0.1524" layer="91"/>
 <wire x1="360.68" y1="139.7" x2="360.68" y2="134.62" width="0.1524" layer="91"/>
@@
 <net name="N$67" class="0">
 <segment>
-<pinref part="V-OCT1" gate="G$1" pin="3"/>
+<pinref part="V-OCT" gate="G$1" pin="3"/>
 <pinref part="R59" gate="G$1" pin="1"/>
 <wire x1="76.2" y1="30.48" x2="88.9" y2="30.48" width="0.1524" layer="91"/>
@@
 <net name="N$9" class="0">
 <segment>
-<pinref part="RES-2" gate="G$1" pin="2"/>
+<pinref part="RES" gate="G$1" pin="2"/>
 <wire x1="233.68" y1="10.16" x2="246.38" y2="10.16" width="0.1524" layer="91"/>
 <wire x1="246.38" y1="10.16" x2="246.38" y2="2.54" width="0.1524" layer="91"/>
@@
 <net name="N$78" class="0">
 <segment>
-<pinref part="RES-2" gate="G$1" pin="3"/>
+<pinref part="RES" gate="G$1" pin="3"/>
 <wire x1="233.68" y1="12.7" x2="254" y2="12.7" width="0.1524" layer="91"/>
 <pinref part="D3" gate="G$1" pin="A"/>
@@
 <segment>
 <pinref part="R79" gate="G$1" pin="1"/>
-<pinref part="IN_MIX" gate="G$1" pin="3"/>
+<pinref part="INPUT_MIX" gate="G$1" pin="3"/>
 <wire x1="370.84" y1="144.78" x2="373.38" y2="144.78" width="0.1524" layer="91"/>
 </segment>
@@
 <segment>
 <pinref part="R9" gate="G$1" pin="1"/>
-<pinref part="IC5" gate="A" pin="OUT"/>
 <wire x1="63.5" y1="-5.08" x2="55.88" y2="-5.08" width="0.1524" layer="91"/>
 <wire x1="55.88" y1="-5.08" x2="55.88" y2="10.16" width="0.1524" layer="91"/>
-<junction x="55.88" y="-5.08"/>
 <pinref part="R6" gate="G$1" pin="2"/>
 <wire x1="55.88" y1="10.16" x2="50.8" y2="10.16" width="0.1524" layer="91"/>
@@
 <pinref part="R8" gate="G$1" pin="2"/>
 <wire x1="35.56" y1="10.16" x2="35.56" y2="-2.54" width="0.1524" layer="91"/>
-<pinref part="IC5" gate="A" pin="-IN"/>
 <wire x1="35.56" y1="-2.54" x2="40.64" y2="-2.54" width="0.1524" layer="91"/>
 <junction x="35.56" y="-2.54"/>
@@
 <wire x1="20.32" y1="-17.78" x2="35.56" y2="-17.78" width="0.1524" layer="91"/>
 <wire x1="35.56" y1="-17.78" x2="35.56" y2="-7.62" width="0.1524" layer="91"/>
-<pinref part="IC5" gate="A" pin="+IN"/>
 <wire x1="35.56" y1="-7.62" x2="40.64" y2="-7.62" width="0.1524" layer="91"/>
 </segment>
@@
 <attribute name="VALUE" x="68.58" y="76.2" size="1.778" layer="96" rot="MR180"/>
 </instance>
+<instance part="IC5" gate="B" x="109.22" y="83.82" smashed="yes">
+<attribute name="NAME" x="111.76" y="80.645" size="1.778" layer="95" rot="MR180"/>
+<attribute name="VALUE" x="111.76" y="88.9" size="1.778" layer="96" rot="MR180"/>
+</instance>
+<instance part="OUTPUT2" gate="G$1" x="154.94" y="91.44" smashed="yes">
+<attribute name="NAME" x="152.4" y="95.504" size="1.778" layer="95"/>
+</instance>
+<instance part="GND7" gate="1" x="147.32" y="83.82" smashed="yes" rot="MR0">
+<attribute name="VALUE" x="149.86" y="81.28" size="1.778" layer="96" rot="MR0"/>
+</instance>
+<instance part="R10" gate="G$1" x="139.7" y="93.98" smashed="yes">
+<attribute name="NAME" x="135.89" y="95.4786" size="1.778" layer="95"/>
+<attribute name="VALUE" x="135.89" y="90.678" size="1.778" layer="96"/>
+</instance>
 </instances>
 <busses>
@@
 <pinref part="OUTPUTLEVEL" gate="G$1" pin="1"/>
 <wire x1="91.44" y1="50.8" x2="91.44" y2="45.72" width="0.1524" layer="91"/>
+</segment>
+<segment>
+<pinref part="GND7" gate="1" pin="GND"/>
+<wire x1="147.32" y1="86.36" x2="147.32" y2="88.9" width="0.1524" layer="91"/>
+<pinref part="OUTPUT2" gate="G$1" pin="1"/>
+<wire x1="147.32" y1="88.9" x2="149.86" y2="88.9" width="0.1524" layer="91"/>
 </segment>
 </net>
@@
 </segment>
 </net>
-<net name="N$4" class="0">
-<segment>
+<net name="N$10" class="0">
+<segment>
+<pinref part="IC5" gate="B" pin="-IN"/>
+<wire x1="101.6" y1="86.36" x2="96.52" y2="86.36" width="0.1524" layer="91"/>
+<wire x1="96.52" y1="86.36" x2="96.52" y2="93.98" width="0.1524" layer="91"/>
+<wire x1="96.52" y1="93.98" x2="124.46" y2="93.98" width="0.1524" layer="91"/>
+<wire x1="124.46" y1="93.98" x2="124.46" y2="83.82" width="0.1524" layer="91"/>
+<pinref part="IC5" gate="B" pin="OUT"/>
+<wire x1="116.84" y1="83.82" x2="124.46" y2="83.82" width="0.1524" layer="91"/>
+</segment>
+</net>
+<net name="N$11" class="0">
+<segment>
+<pinref part="IC5" gate="B" pin="+IN"/>
+<wire x1="101.6" y1="81.28" x2="96.52" y2="81.28" width="0.1524" layer="91"/>
 <wire x1="96.52" y1="55.88" x2="106.68" y2="55.88" width="0.1524" layer="91"/>
 <pinref part="R57" gate="G$1" pin="1"/>
 <pinref part="OUTPUTLEVEL" gate="G$1" pin="2"/>
-</segment>
-</net>
+<wire x1="96.52" y1="81.28" x2="96.52" y2="55.88" width="0.1524" layer="91"/>
+<junction x="96.52" y="55.88"/>
+</segment>
+</net>
+<net name="O1" class="0">
+<segment>
+<pinref part="R10" gate="G$1" pin="2"/>
+<pinref part="OUTPUT2" gate="G$1" pin="3"/>
+<wire x1="144.78" y1="93.98" x2="149.86" y2="93.98" width="0.1524" layer="91"/>
+</segment>
+</net>
+<net name="N$14" class="0">
+<segment>
+<wire x1="124.46" y1="93.98" x2="134.62" y2="93.98" width="0.1524" layer="91"/>
+<pinref part="R10" gate="G$1" pin="1"/>
+</segment>
+</net>
